File: board/board.kicad_pcb (KiCad board)
At the start: 2 copper layers, 21 x 13 mm, 1 part

Commit message: initial
Parts:
- removed LOGO1: Logo_Open_Hardware_Small, Symbol:OSHW-Symbol_6.7x6mm_SilkScreen
- added J1: 020_1000BASE-T_with_CT, on_edge:on_edge_2x10_device, F.Cu at (50.0, 142.0)
- added J2: 004_BASE-T_CT, on_edge:on_edge_2x05_host, F.Cu at (74.0, 159.0)
- added R1: d.n.p, Resistor_SMD:R_1206_3216Metric, F.Cu at (66.4, 156.5)
- added U1: MagJack-A70-112-331N126, b086:TRJG0926HENL, F.Cu at (68.0, 145.4)
- added l1: Logo_Open_Hardware_Larg, Symbol:OSHW-Logo2_7.3x6mm_SilkScreen, F.Cu at (65.5, 160.5)
Routing:
- net GND: track 0.00 -> 42.1 mm, vias 0 -> 3
- net Net-(J1-Pad14): track 0.00 -> 30.7 mm, vias 0 -> 2
- net Net-(J1-Pad15): track 0.00 -> 30.3 mm, vias 0 -> 2
- net /TR3_TAP: track 0.00 -> 26.9 mm
- net /TRD3_N: track 0.00 -> 26.0 mm, vias 0 -> 1
- net Net-(J1-Pad19): track 0.00 -> 26.0 mm, vias 0 -> 1
- net /TRD3_P: track 0.00 -> 25.6 mm, vias 0 -> 1
- net Net-(J1-Pad6): track 0.00 -> 23.9 mm, vias 0 -> 1
- net Net-(J1-Pad20): track 0.00 -> 23.4 mm, vias 0 -> 1
- net Net-(J1-Pad16): track 0.00 -> 22.7 mm, vias 0 -> 1
- net /TR1_TAP: track 0.00 -> 21.2 mm
- net Net-(R1-Pad1): track 0.00 -> 20.7 mm
- net /TR2_TAP: track 0.00 -> 19.2 mm
- net /TRD0_N: track 0.00 -> 18.4 mm
- net /TRD1_N: track 0.00 -> 17.8 mm, vias 0 -> 1
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Other:
- board size 21 x 13 mm -> 24 x 29 mm
- copper layers 2 -> 4
- rule pad_to_mask_clearance: 0 -> 0.04
- board text added: "osf.004"
- board text added: "osf.020"
- board text added: "osf.b086.v1.0"
